File: Hardware/E-Book Reader.brd (EAGLE design)
At the start: 170.3 x 111.4 mm, 103 parts, among them IC1 BD5229G-TR, IC4 XC6220A331MR-G, J1 FH34SRJ-24S-0.5SH_99_, J2 SAMACSYS_PARTS_USB4110-GF-A, J3 QWIIC_RIGHT_ANGLE, J4 112A-TAAR-R03_ATTEND, Q1 20V/4.2A/52mΩ/1.4W, Q2 20V/4.2A/52mΩ/1.4W, Q3 SI1308EDL-T1-GE3, U1 MAX17048G+T10, U2 ESP32-C6-WROOM-1-N8, U3 W25Q512JVEIQ, U4 DS3231SN#

Commit message: Updated Schematic and PCB After Fixing Issues
Parts:
- moved R2-USB 0.76 mm to (155.8, 51.6)
- renumbered TP1 to TP_TX, TP10 to TP_EPD_CS, TP11 to TP_EPD_DC, TP12 to TP_EPD_RST, TP13 to TP_3V3_C, TP14 to TP_VBUS, TP15 to TP_INT_RTC, TP16 to TP_3V3, TP17 to TP_EPD_3V3, TP2 to TP_RX, TP3 to TP_VBAT, TP4 to TP_GND1, TP5 to TP_GND, TP6 to TP_MISO, TP7 to TP_MOSI, TP8 to TP_SCK, TP9 to TP_EPD_BUSY
Routing:
- net SS_SD: track 93.9 -> 96.3 mm
- net VUSB: track 35.2 -> 32.9 mm
- net MOSI: track 193.2 -> 191.5 mm
- net 3V3: track 408.7 -> 407.1 mm
- net PREVGL: track 86.6 -> 85.5 mm
- net EPD_RST: track 130.0 -> 131.1 mm
- net P_NET_18: track 8.85 -> 7.97 mm
- net 32KHZ: track 85.9 -> 86.7 mm
- net SCK: track 166.2 -> 167.0 mm
- net DN: track 14.0 -> 13.3 mm
- net EPD_BUSY: track 137.9 -> 138.6 mm
- net EPD_CS: track 178.7 -> 179.3 mm
- net FLASH_CS: track 128.7 -> 129.2 mm
